File: my_mg10/my_mg10.kicad_pcb (KiCad board)
At the start: 2 copper layers, 270 x 70 mm, 127 parts, among them J1 INPUT, J2 PWR_CONN, J3 AUX INPUT, J4 SEND, J5 RETURN, J6 HEADPHONES, K1 G6S-2, SW1 Clean/Overdrive, SW2 FOOTSWITCH, U1 TL072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

Commit message: Minor file tweaks
Routing:
- net Net-(C32-Pad2): track 148.8 -> 154.5 mm
Changed lines of the file:
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@@
+	)
+	(segment
+		(start 124 111.5)
+		(end 124 108.84)
+		(width 0.6)
+		(layer "F.Cu")
+		(net 34)
+	)
+	(segment
+		(start 124 108.84)
+		(end 121.86 106.7)
+		(width 0.6)
+		(layer "F.Cu")
+		(net 34)
 	)
 	(segment

Commit message: Added headphone out switching, added pictures
Parts:
- removed TP17: HEADPHONES_OUT, TestPoint:TestPoint_THTPad_D2.5mm_Drill1.2mm
- added D11: 1N4007, Diode_THT:D_DO-41_SOD81_P10.16mm_Horizontal, F.Cu at (223.9, 70.6)
- added JP10: ~, TestPoint:TestPoint_2Pads_Pitch2.54mm_Drill0.8mm, F.Cu at (228.4, 63.4)
- added JP11: ~, TestPoint:TestPoint_2Pads_Pitch2.54mm_Drill0.8mm, F.Cu at (254.8, 75.7)
- added JP12: ~, TestPoint:TestPoint_2Pads_Pitch2.54mm_Drill0.8mm, F.Cu at (251.3, 73.2)
- added JP13: ~, TestPoint:TestPoint_2Pads_Pitch2.54mm_Drill0.8mm, F.Cu at (258.2, 73.2)
- added JP9: ~, TestPoint:TestPoint_2Pads_Pitch2.54mm_Drill0.8mm, F.Cu at (59.6, 101.0)
- added K2: G6S-2, Relay_THT:Relay_DPDT_Omron_G6S-2, F.Cu at (232.4, 68.5)
- added R43: R, Resistor_THT:R_Axial_DIN0207_L6.3mm_D2.5mm_P7.62mm_Horizontal, F.Cu at (261.5, 99.0)
- added TP4: +5V_TP, TestPoint:TestPoint_THTPad_D2.5mm_Drill1.2mm, F.Cu at (161.6, 82.4)
- moved LS1 27.4 mm to (253.7, 65.0)
- moved R36 11.0 mm to (261.5, 95.0), turned to 180 degrees
- moved TP2 4.80 mm to (153.2, 82.5)
Connections:
- J6 pad SN: unconnected-(J6-PadSN) -> Net-(JP10-B)
- LS1 pad 1: Net-(D10-K) -> Net-(K2-Pad8)
- R36 pad 1: Net-(D10-K) -> Net-(C40-Pad1)
- R36 pad 2: Net-(C40-Pad1) -> Net-(K2-Pad10)
- R41 pad 2: Net-(D1-A) -> Net-(JP9-B)
- R42 pad 2: Net-(D1-A) -> Net-(JP9-B)
- SW1 pad 2: Net-(D1-A) -> Net-(JP9-B)
- SW2 pad 2: Net-(D1-A) -> Net-(JP9-B)
Routing:
- net +5V: track 125.3 -> 239.4 mm
- net Net-(JP10-B): track 0.00 -> 91.8 mm
- net Net-(D1-A): track 96.3 -> 27.2 mm
- net Net-(JP9-B): track 0.00 -> 66.4 mm
- net Net-(K2-Pad10): track 0.00 -> 54.0 mm
- net Net-(D10-K): track 114.0 -> 88.4 mm
- net +15V: track 351.6 -> 370.1 mm
- net Net-(JP13-A): track 0.00 -> 17.5 mm
- net Net-(JP11-B): track 0.00 -> 16.6 mm
- net Net-(JP12-A): track 0.00 -> 15.7 mm
- net Net-(K2-Pad8): track 0.00 -> 11.7 mm
- net Net-(D11-A): track 0.00 -> 9.79 mm
- net Net-(LS1-Pad2): track 94.1 -> 100.0 mm
- net Net-(C40-Pad1): track 27.8 -> 29.2 mm
Other:
- board text added: "+5V"
